Commit message: chore(release): v1.0.0 for WSL
Adds all-in-one bash launch script, daemonizes MAVProxy, fixes OpenCV compatibility and standardizes ArUco dict.

File: models/husky/urdf/ugv.urdf.xacro (robot description, xacro)
@@ -6,10 +6,10 @@
       <cast_shadows>true</cast_shadows>
       <geometry>
-        <mesh filename="package://mp_uav_landing_sim/models/husky/meshes/platform.dae" scale="0.5 0.5 0.5"/>
-      </geometry>
-    </visual>
-    <collision>
-      <geometry>
-        <mesh filename="package://mp_uav_landing_sim/models/husky/meshes/platform.dae" scale="0.5 0.5 0.5"/>
+        <mesh filename="package://arkhe_gazebo/models/husky/meshes/platform.dae" scale="0.5 0.5 0.5"/>
+      </geometry>
+    </visual>
+    <collision>
+      <geometry>
+        <mesh filename="package://arkhe_gazebo/models/husky/meshes/platform.dae" scale="0.5 0.5 0.5"/>
       </geometry>
     </collision>
@@ -24,10 +24,10 @@
       <cast_shadows>true</cast_shadows>
       <geometry>
-        <mesh filename="package://mp_uav_landing_sim/models/husky/meshes/uwb_anchor.dae" scale="1 1 1"/>
-      </geometry>
-    </visual>
-    <collision>
-      <geometry>
-        <mesh filename="package://mp_uav_landing_sim/models/husky/meshes/uwb_anchor.dae" scale="1 1 1"/>
+        <mesh filename="package://arkhe_gazebo/models/husky/meshes/uwb_anchor.dae" scale="1 1 1"/>
+      </geometry>
+    </visual>
+    <collision>
+      <geometry>
+        <mesh filename="package://arkhe_gazebo/models/husky/meshes/uwb_anchor.dae" scale="1 1 1"/>
       </geometry>
     </collision>
@@ -42,10 +42,10 @@
       <cast_shadows>true</cast_shadows>
       <geometry>
-        <mesh filename="package://mp_uav_landing_sim/models/husky/meshes/uwb_anchor.dae" scale="1 1 1"/>
-      </geometry>
-    </visual>
-    <collision>
-      <geometry>
-        <mesh filename="package://mp_uav_landing_sim/models/husky/meshes/uwb_anchor.dae" scale="1 1 1"/>
+        <mesh filename="package://arkhe_gazebo/models/husky/meshes/uwb_anchor.dae" scale="1 1 1"/>
+      </geometry>
+    </visual>
+    <collision>
+      <geometry>
+        <mesh filename="package://arkhe_gazebo/models/husky/meshes/uwb_anchor.dae" scale="1 1 1"/>
       </geometry>
     </collision>
@@ -60,10 +60,10 @@
       <cast_shadows>true</cast_shadows>
       <geometry>
-        <mesh filename="package://mp_uav_landing_sim/models/husky/meshes/uwb_anchor.dae" scale="1 1 1"/>
-      </geometry>
-    </visual>
-    <collision>
-      <geometry>
-        <mesh filename="package://mp_uav_landing_sim/models/husky/meshes/uwb_anchor.dae" scale="1 1 1"/>
+        <mesh filename="package://arkhe_gazebo/models/husky/meshes/uwb_anchor.dae" scale="1 1 1"/>
+      </geometry>
+    </visual>
+    <collision>
+      <geometry>
+        <mesh filename="package://arkhe_gazebo/models/husky/meshes/uwb_anchor.dae" scale="1 1 1"/>
       </geometry>
     </collision>
@@ -78,10 +78,10 @@
       <cast_shadows>true</cast_shadows>
       <geometry>
-        <mesh filename="package://mp_uav_landing_sim/models/husky/meshes/uwb_anchor.dae" scale="1 1 1"/>
-      </geometry>
-    </visual>
-    <collision>
-      <geometry>
-        <mesh filename="package://mp_uav_landing_sim/models/husky/meshes/uwb_anchor.dae" scale="1 1 1"/>
+        <mesh filename="package://arkhe_gazebo/models/husky/meshes/uwb_anchor.dae" scale="1 1 1"/>
+      </geometry>
+    </visual>
+    <collision>
+      <geometry>
+        <mesh filename="package://arkhe_gazebo/models/husky/meshes/uwb_anchor.dae" scale="1 1 1"/>
       </geometry>
     </collision>
@@ -96,10 +96,10 @@
       <cast_shadows>true</cast_shadows>
       <geometry>
-        <mesh filename="package://mp_uav_landing_sim/models/husky/meshes/marker.dae" />
-      </geometry>
-    </visual>
-    <collision>
-      <geometry>
-        <mesh filename="package://mp_uav_landing_sim/models/husky/meshes/marker.dae" />
+        <mesh filename="package://arkhe_gazebo/models/husky/meshes/marker.dae" />
+      </geometry>
+    </visual>
+    <collision>
+      <geometry>
+        <mesh filename="package://arkhe_gazebo/models/husky/meshes/marker.dae" />
       </geometry>
     </collision>
@@ -114,10 +114,10 @@
       <cast_shadows>true</cast_shadows>
       <geometry>
-        <mesh filename="package://mp_uav_landing_sim/models/husky/meshes/diode.dae" scale="0.4 0.4 0.4"/>
-      </geometry>
-    </visual>
-    <collision>
-      <geometry>
-        <mesh filename="package://mp_uav_landing_sim/models/husky/meshes/diode.dae" scale="0.4 0.4 0.4"/>
+        <mesh filename="package://arkhe_gazebo/models/husky/meshes/diode.dae" scale="0.4 0.4 0.4"/>
+      </geometry>
+    </visual>
+    <collision>
+      <geometry>
+        <mesh filename="package://arkhe_gazebo/models/husky/meshes/diode.dae" scale="0.4 0.4 0.4"/>
       </geometry>
     </collision>
@@ -132,10 +132,10 @@
       <cast_shadows>true</cast_shadows>
       <geometry>
-        <mesh filename="package://mp_uav_landing_sim/models/husky/meshes/diode.dae" scale="0.4 0.4 0.4"/>
-      </geometry>
-    </visual>
-    <collision>
-      <geometry>
-        <mesh filename="package://mp_uav_landing_sim/models/husky/meshes/diode.dae" scale="0.4 0.4 0.4"/>
+        <mesh filename="package://arkhe_gazebo/models/husky/meshes/diode.dae" scale="0.4 0.4 0.4"/>
+      </geometry>
+    </visual>
+    <collision>
+      <geometry>
+        <mesh filename="package://arkhe_gazebo/models/husky/meshes/diode.dae" scale="0.4 0.4 0.4"/>
       </geometry>
     </collision>
@@ -150,10 +150,10 @@
       <cast_shadows>true</cast_shadows>
       <geometry>
-        <mesh filename="package://mp_uav_landing_sim/models/husky/meshes/diode.dae" scale="0.4 0.4 0.4"/>
-      </geometry>
-    </visual>
-    <collision>
-      <geometry>
-        <mesh filename="package://mp_uav_landing_sim/models/husky/meshes/diode.dae" scale="0.4 0.4 0.4"/>
+        <mesh filename="package://arkhe_gazebo/models/husky/meshes/diode.dae" scale="0.4 0.4 0.4"/>
+      </geometry>
+    </visual>
+    <collision>
+      <geometry>
+        <mesh filename="package://arkhe_gazebo/models/husky/meshes/diode.dae" scale="0.4 0.4 0.4"/>
       </geometry>
     </collision>
@@ -168,10 +168,10 @@
       <cast_shadows>true</cast_shadows>
       <geometry>
-        <mesh filename="package://mp_uav_landing_sim/models/husky/meshes/diode.dae" scale="0.4 0.4 0.4"/>
-      </geometry>
-    </visual>
-    <collision>
-      <geometry>
-        <mesh filename="package://mp_uav_landing_sim/models/husky/meshes/diode.dae" scale="0.4 0.4 0.4"/>
+        <mesh filename="package://arkhe_gazebo/models/husky/meshes/diode.dae" scale="0.4 0.4 0.4"/>
+      </geometry>
+    </visual>
+    <collision>
+      <geometry>
+        <mesh filename="package://arkhe_gazebo/models/husky/meshes/diode.dae" scale="0.4 0.4 0.4"/>
       </geometry>
     </collision>

Commit message: feat(sim): Add headless mode, shrink ArUco marker to 0.21m and update pose controller

File: models/husky/urdf/ugv.urdf.xacro (robot description, xacro)
@@ -96,10 +96,10 @@
       <cast_shadows>true</cast_shadows>
       <geometry>
-        <mesh filename="package://arkhe_gazebo/models/husky/meshes/marker.dae" />
-      </geometry>
-    </visual>
-    <collision>
-      <geometry>
-        <mesh filename="package://arkhe_gazebo/models/husky/meshes/marker.dae" />
+        <mesh filename="package://arkhe_gazebo/models/husky/meshes/marker.dae" scale="0.2 0.2 1.0"/>
+      </geometry>
+    </visual>
+    <collision>
+      <geometry>
+        <mesh filename="package://arkhe_gazebo/models/husky/meshes/marker.dae" scale="0.2 0.2 1.0"/>
       </geometry>
     </collision>
